File: LH_RKJXM1015004_FacePlateTilted/LH_RKJXM1015004_FacePlateTilted.kicad_pcb (KiCad board)
At the start: 2 copper layers, 21.1 x 17.3 mm, 3 parts, among them U1 RKJXM1015004

Commit message: library fix
Parts:
- U1: footprint MyLibrary:RKJXM1015004 -> Alps:RKJXM1015004
Connections:
- U1 pad 1: Net-(U1-Pad1) -> unconnected-(U1-GND-Pad1)
- U1 pad 2: Net-(U1-Pad2) -> unconnected-(U1-PUSH-Pad2)
- U1 pad 3: Net-(U1-Pad3) -> unconnected-(U1-COM-Pad3)
- U1 pad 4: Net-(U1-Pad4) -> unconnected-(U1-A-Pad4)
- U1 pad 5: Net-(U1-Pad5) -> unconnected-(U1-B-Pad5)
- U1 pad 6: Net-(J1-Pad5) -> unconnected-(U1-C-Pad6)
- U1 pad 7: Net-(U1-Pad7) -> unconnected-(U1-D-Pad7)
Routing:
- net unconnected-(U1-PUSH-Pad2): track 0.00 -> 16.3 mm
- net Net-(U1-Pad2): track 16.3 -> 0.00 mm
Changed lines of the file:
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@@
   )
   (net 0 "")
-  (net 1 "Net-(J1-Pad5)")
-  (net 2 "Net-(U1-Pad1)")
-  (net 3 "Net-(U1-Pad2)")
-  (net 4 "Net-(U1-Pad3)")
-  (net 5 "Net-(U1-Pad7)")
-  (net 6 "Net-(U1-Pad5)")
-  (net 7 "Net-(U1-Pad4)")
+  (net 1 "unconnected-(U1-GND-Pad1)")
+  (net 2 "unconnected-(U1-PUSH-Pad2)")
+  (net 3 "unconnected-(U1-COM-Pad3)")
+  (net 4 "unconnected-(U1-A-Pad4)")
+  (net 5 "unconnected-(U1-B-Pad5)")
+  (net 6 "unconnected-(U1-C-Pad6)")
+  (net 7 "unconnected-(U1-D-Pad7)")
   (footprint "MountingHole:MountingHole_2.2mm_M2" (layer "F.Cu")
     (at 43.772759 61.75)
@@
     (pad "" np_thru_hole circle (at 0 0) (size 2.2 2.2) (drill 2.2) (layers "*.Cu" "*.Mask"))
   )
-  (footprint "MyLibrary:RKJXM1015004" (layer "B.Cu")
+  (footprint "Alps:RKJXM1015004" (layer "B.Cu")
     (at 52 57 180)
-    (property "Sheetfile" "RH_RKJXM1015004_FacePlateTilted.kicad_sch")
+    (property "Sheetfile" "LH_RKJXM1015004_FacePlateTilted.kicad_sch")
     (property "Sheetname" "")
     (attr through_hole)
-    (fp_text reference "U1" (at 0 0.5 unlocked) (layer "B.SilkS") hide
+    (fp_text reference "U1" (at 0 0.499999 unlocked) (layer "B.SilkS") hide
         (effects (font (size 1 1) (thickness 0.15)) (justify mirror))
     )
@@
         (effects (font (size 0.5 0.5) (thickness 0.1)))
     )
-    (fp_text user "B" (at 3.7 1 unlocked) (layer "F.SilkS")
+    (fp_text user "PUSH" (at -1 -4 unlocked) (layer "F.SilkS")
+        (effects (font (size 0.5 0.5) (thickness 0.1)))
+    )
+    (fp_text user "GND" (at -2.35 2.78 unlocked) (layer "F.SilkS")
         (effects (font (size 0.5 0.5) (thickness 0.1)))
     )
@@
         (effects (font (size 0.5 0.5) (thickness 0.1)))
     )
-    (fp_text user "PUSH" (at -3.4 1 unlocked) (layer "F.SilkS")
+    (fp_text user "B" (at 3.7 1 unlocked) (layer "F.SilkS")
+        (effects (font (size 0.5 0.5) (thickness 0.1)))
+    )
+    (fp_text user "C" (at -1 3.6 unlocked) (layer "F.SilkS")
+        (effects (font (size 0.5 0.5) (thickness 0.1)))
+    )
+    (fp_text user "D" (at -3.7 -1 unlocked) (layer "F.SilkS")
         (effects (font (size 0.5 0.5) (thickness 0.1)))
     )
@@
         (effects (font (size 0.5 0.5) (thickness 0.1)))
     )
-    (fp_text user "D" (at -3.7 -1 unlocked) (layer "F.SilkS")
-        (effects (font (size 0.5 0.5) (thickness 0.1)))
-    )
-    (fp_text user "GND" (at -2.35 2.78 unlocked) (layer "F.SilkS")
-        (effects (font (size 0.5 0.5) (thickness 0.1)))
-    )
-    (fp_text user "PUSH" (at -1 -4 unlocked) (layer "F.SilkS")
-        (effects (font (size 0.5 0.5) (thickness 0.1)))
-    )
-    (fp_text user "C" (at -1 3.6 unlocked) (layer "F.SilkS")
+    (fp_text user "PUSH" (at -3.4 1 unlocked) (layer "F.SilkS")
         (effects (font (size 0.5 0.5) (thickness 0.1)))
     )
@@
     (pad "" np_thru_hole circle (at 1 3 180) (size 1.1 1.1) (drill 1.1) (layers "F&B.Cu" "*.Mask"))
     (pad "1" thru_hole circle (at -4.15 2.7 180) (size 1.6 1.6) (drill 1) (layers "*.Cu" "*.Mask")
-      (net 2 "Net-(U1-Pad1)") (pinfunction "GND") (pintype "power_out"))
+      (net 1 "unconnected-(U1-GND-Pad1)") (pinfunction "GND") (pintype "power_out"))
     (pad "2" thru_hole circle (at -5.35 1 180) (size 1.6 1.6) (drill 1) (layers "*.Cu" "*.Mask")
-      (net 3 "Net-(U1-Pad2)") (pinfunction "PUSH") (pintype "power_in"))
+      (net 2 "unconnected-(U1-PUSH-Pad2)") (pinfunction "PUSH") (pintype "power_in"))
     (pad "2" thru_hole circle (at -1 -5.35 180) (size 1.6 1.6) (drill 1) (layers "*.Cu" "*.Mask")
-      (net 3 "Net-(U1-Pad2)") (pinfunction "PUSH") (pintype "power_in"))
+      (net 2 "unconnected-(U1-PUSH-Pad2)") (pinfunction "PUSH") (pintype "power_in"))
     (pad "2" thru_hole circle (at 5.35 -1 180) (size 1.6 1.6) (drill 1) (layers "*.Cu" "*.Mask")
-      (net 3 "Net-(U1-Pad2)") (pinfunction "PUSH") (pintype "power_in"))
+      (net 2 "unconnected-(U1-PUSH-Pad2)") (pinfunction "PUSH") (pintype "power_in"))
     (pad "3" thru_hole circle (at 1 5.35 180) (size 1.6 1.6) (drill 1) (layers "*.Cu" "*.Mask")
-      (net 4 "Net-(U1-Pad3)") (pinfunction "COM") (pintype "output"))
+      (net 3 "unconnected-(U1-COM-Pad3)") (pinfunction "COM") (pintype "output"))
     (pad "4" thru_hole circle (at 1 -4.95 180) (size 1.6 1.6) (drill 1) (layers "*.Cu" "*.Mask")
-      (net 7 "Net-(U1-Pad4)") (pinfunction "A") (pintype "output"))
+      (net 4 "unconnected-(U1-A-Pad4)") (pinfunction "A") (pintype "output"))
     (pad "5" thru_hole circle (at 4.95 1 180) (size 1.6 1.6) (drill 1) (layers "*.Cu" "*.Mask")
-      (net 6 "Net-(U1-Pad5)") (pinfunction "B") (pintype "output"))
+      (net 5 "unconnected-(U1-B-Pad5)") (pinfunction "B") (pintype "output"))
     (pad "6" thru_hole circle (at -1 4.95 180) (size 1.6 1.6) (drill 1) (layers "*.Cu" "*.Mask")
-      (net 1 "Net-(J1-Pad5)") (pinfunction "C") (pintype "output"))
+      (net 6 "unconnected-(U1-C-Pad6)") (pinfunction "C") (pintype "output"))
     (pad "7" thru_hole circle (at -4.95 -1 180) (size 1.6 1.6) (drill 1) (layers "*.Cu" "*.Mask")
-      (net 5 "Net-(U1-Pad7)") (pinfunction "D") (pintype "output"))
-    (model "V:/ECAD/MyCustomLibrary/3D/MultiDirectionSwitch/RKJXM1015004.step"
+      (net 7 "unconnected-(U1-D-Pad7)") (pinfunction "D") (pintype "output"))
+    (model "../libraries/Alps_kicadlib/Alps.3dshapes/RKJXM1015004.STEP"
       (offset (xyz 0 0 0))
       (scale (xyz 1 1 1))
-      (rotate (xyz 0 0 0))
+      (rotate (xyz 0 -180 0))
     )
   )
@@
   (gr_line (start 60.988764 48.311458) (end 58.831 50.3957)
     (stroke (width 0.1) (type solid)) (layer "User.1"))
-  (segment (start 53 58.9) (end 53.9 58) (width 0.25) (layer "B.Cu") (net 3))
-  (segment (start 53 62.35) (end 53 58.9) (width 0.25) (layer "B.Cu") (net 3))
-  (segment (start 55.9 56) (end 57.35 56) (width 0.25) (layer "B.Cu") (net 3))
-  (segment (start 53.9 58) (end 55.9 56) (width 0.25) (layer "B.Cu") (net 3))
-  (segment (start 46.65 58) (end 53.9 58) (width 0.25) (layer "B.Cu") (net 3))
-  (segment (start 47.075 56) (end 46.65 56) (width 0.5) (layer "F.Cu") (net 6))
+  (segment (start 53 58.9) (end 53.9 58) (width 0.25) (layer "B.Cu") (net 2))
+  (segment (start 53 62.35) (end 53 58.9) (width 0.25) (layer "B.Cu") (net 2))
+  (segment (start 55.9 56) (end 57.35 56) (width 0.25) (layer "B.Cu") (net 2))
+  (segment (start 53.9 58) (end 55.9 56) (width 0.25) (layer "B.Cu") (net 2))
+  (segment (start 46.65 58) (end 53.9 58) (width 0.25) (layer "B.Cu") (net 2))
+  (segment (start 47.075 56) (end 46.65 56) (width 0.5) (layer "F.Cu") (net 5))
 )
