File: LH_RKJXM1015004_FacePlateTilted/LH_RKJXM1015004_FacePlateTilted.kicad_sch (KiCad schematic)
At the start: 1 part, among them U1 RKJXM1015004

Commit message: library fix
Parts:
- U1: footprint MyLibrary:RKJXM1015004 -> Alps:RKJXM1015004; symbol MyLibrary:RKJXM1015004 -> Alps:RKJXM1015004
Other:
- moved on the sheet: U1
Changed lines of the file:
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@@
-(kicad_sch (version 20211123) (generator eeschema)
+(kicad_sch (version 20230121) (generator eeschema)
   (paper "A4")
-  (symbol (lib_id "MyLibrary:RKJXM1015004") (at 64.77 53.34 0) (unit 1)
-    (in_bom yes) (on_board yes) (fields_autoplaced)
-    (property "Reference" "U1" (id 0) (at 64.135 35.56 0))
-    (property "Value" "RKJXM1015004" (id 1) (at 64.135 38.1 0))
-    (property "Footprint" "MyLibrary:RKJXM1015004" (id 2) (at 64.77 53.34 0)
+  (symbol (lib_id "Alps:RKJXM1015004") (at 64.77 53.34 0) (unit 1)
+    (in_bom yes) (on_board yes) (dnp no) (fields_autoplaced)
+    (property "Reference" "U1" (at 64.135 35.56 0)
+      (effects (font (size 1.27 1.27)))
+    )
+    (property "Value" "RKJXM1015004" (at 64.135 38.1 0)
+      (effects (font (size 1.27 1.27)))
+    )
+    (property "Footprint" "Alps:RKJXM1015004" (at 64.77 53.34 0)
       (effects (font (size 1.27 1.27)) hide)
     )
-    (property "Datasheet" "" (id 3) (at 64.77 53.34 0)
+    (property "Datasheet" "" (at 64.77 53.34 0)
       (effects (font (size 1.27 1.27)) hide)
     )
@@
     (pin "6")
     (pin "7")
+    (instances
+      (project "LH_RKJXM1015004_FacePlateTilted"
+        (path "/ff8ac8c3-4f7d-424b-9e6e-e056f231a7a0"
+          (reference "U1") (unit 1)
+        )
+      )
+    )
   )
   (sheet_instances
     (path "/" (page "1"))
   )
-  (symbol_instances
-    (path "/5b54b85c-0d1c-400d-ad5f-62ef31771a21"
-      (reference "U1") (unit 1) (value "RKJXM1015004") (footprint "MyLibrary:RKJXM1015004")
-    )
-  )
 )
