File: RH_BreakLever_FreeJoy/RH_BreakLever_FreeJoy.kicad_pcb (KiCad board)
At the start: 2 copper layers, 36.4 x 16.3 mm, 5 parts, among them J1 Conn_01x06, M1 MountingHole_2.2mm_M2, M2 MountingHole_2.2mm_M2, U1 SS495A, U2 MCP3201

Commit message: updated a footprint on Break-lever design for footprint naming.
Parts:
- J1: value Conn_01x06 -> Conn_01x05
- U2: footprint Package_SO:PowerIntegrations_SO-8 -> Package_SO:SOIC-8_3.9x4.9mm_P1.27mm
Changed lines of the file:
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@@
         (effects (font (size 1 1) (thickness 0.15)))
     )
-    (fp_text value "Conn_01x06" (at 5 4.6 90) (layer "F.Fab")
+    (fp_text value "Conn_01x05" (at 5 4.6 90) (layer "F.Fab")
         (effects (font (size 1 1) (thickness 0.15)))
     )
@@
     )
   )
-  (footprint "Package_SO:PowerIntegrations_SO-8" (layer "B.Cu")
+  (footprint "Package_SO:SOIC-8_3.9x4.9mm_P1.27mm" (layer "B.Cu")
     (at 52.675 24.9 180)
-    (descr "Power-Integrations variant of 8-Lead Plastic Small Outline (SN) - Narrow, 3.90 mm Body [SOIC], see https://ac-dc.power.com/sites/default/files/product-docs/senzero_family_datasheet.pdf")
-    (tags "SOIC 1.27")
+    (descr "SOIC, 8 Pin (JEDEC MS-012AA, https://www.analog.com/media/en/package-pcb-resources/package/pkg_pdf/soic_narrow-r/r_8.pdf), generated with kicad-footprint-generator ipc_gullwing_generator.py")
+    (tags "SOIC SO")
     (property "Sheetfile" "RH_BreakLever_FreeJoy.kicad_sch")
     (property "Sheetname" "")
@@
     (property "ki_keywords" "12-Bit Differential ADC SPI 1ch")
     (attr smd)
-    (fp_text reference "U2" (at 0 -0.5) (layer "B.SilkS")
+    (fp_text reference "U2" (at 0 3.4) (layer "B.SilkS")
         (effects (font (size 1 1) (thickness 0.15)) (justify mirror))
     )
-    (fp_text value "MCP3201" (at 0 -3.5) (layer "B.Fab")
+    (fp_text value "MCP3201" (at 0 -3.4) (layer "B.Fab")
         (effects (font (size 1 1) (thickness 0.15)) (justify mirror))
     )
     (fp_text user "${REFERENCE}" (at 0 0) (layer "B.Fab")
-        (effects (font (size 1 1) (thickness 0.15)) (justify mirror))
+        (effects (font (size 0.98 0.98) (thickness 0.15)) (justify mirror))
     )
-    (fp_line (start -2.075 -2.575) (end -2.075 -2.43)
-      (stroke (width 0.15) (type solid)) (layer "B.SilkS"))
-    (fp_line (start -2.075 -2.575) (end 2.075 -2.575)
-      (stroke (width 0.15) (type solid)) (layer "B.SilkS"))
-    (fp_line (start -2.075 2.525) (end -3.475 2.525)
-      (stroke (width 0.15) (type solid)) (layer "B.SilkS"))
-    (fp_line (start -2.075 2.575) (end -2.075 2.525)
-      (stroke (width 0.15) (type solid)) (layer "B.SilkS"))
-    (fp_line (start -2.075 2.575) (end 2.075 2.575)
-      (stroke (width 0.15) (type solid)) (layer "B.SilkS"))
-    (fp_line (start 2.075 -2.575) (end 2.075 -2.43)
-      (stroke (width 0.15) (type solid)) (layer "B.SilkS"))
-    (fp_line (start 2.075 2.575) (end 2.075 2.43)
-      (stroke (width 0.15) (type solid)) (layer "B.SilkS"))
-    (fp_line (start -3.98 2.7) (end -3.98 -2.7)
+    (fp_line (start 0 -2.56) (end -1.95 -2.56)
+      (stroke (width 0.12) (type solid)) (layer "B.SilkS"))
+    (fp_line (start 0 -2.56) (end 1.95 -2.56)
+      (stroke (width 0.12) (type solid)) (layer "B.SilkS"))
+    (fp_line (start 0 2.56) (end -3.45 2.56)
+      (stroke (width 0.12) (type solid)) (layer "B.SilkS"))
+    (fp_line (start 0 2.56) (end 1.95 2.56)
+      (stroke (width 0.12) (type solid)) (layer "B.SilkS"))
+    (fp_line (start -3.7 -2.7) (end 3.7 -2.7)
       (stroke (width 0.05) (type solid)) (layer "B.CrtYd"))
-    (fp_line (start -3.98 2.7) (end 3.97 2.7)
+    (fp_line (start -3.7 2.7) (end -3.7 -2.7)
       (stroke (width 0.05) (type solid)) (layer "B.CrtYd"))
-    (fp_line (start 3.97 -2.7) (end -3.98 -2.7)
+    (fp_line (start 3.7 -2.7) (end 3.7 2.7)
       (stroke (width 0.05) (type solid)) (layer "B.CrtYd"))
-    (fp_line (start 3.97 -2.7) (end 3.97 2.7)
+    (fp_line (start 3.7 2.7) (end -3.7 2.7)
       (stroke (width 0.05) (type solid)) (layer "B.CrtYd"))
-    (fp_line (start -1.95 -2.45) (end -1.95 1.45)
+    (fp_line (start -1.95 -2.45) (end -1.95 1.475)
       (stroke (width 0.1) (type solid)) (layer "B.Fab"))
-    (fp_line (start -1.95 1.45) (end -0.95 2.45)
+    (fp_line (start -1.95 1.475) (end -0.975 2.45)
       (stroke (width 0.1) (type solid)) (layer "B.Fab"))
-    (fp_line (start -0.95 2.45) (end 1.95 2.45)
+    (fp_line (start -0.975 2.45) (end 1.95 2.45)
       (stroke (width 0.1) (type solid)) (layer "B.Fab"))
     (fp_line (start 1.95 -2.45) (end -1.95 -2.45)
@@
     (fp_line (start 1.95 2.45) (end 1.95 -2.45)
       (stroke (width 0.1) (type solid)) (layer "B.Fab"))
-    (pad "1" smd rect (at -2.725 1.905 180) (size 2 0.6) (layers "B.Cu" "B.Paste" "B.Mask")
+    (pad "1" smd roundrect (at -2.475 1.905 180) (size 1.95 0.6) (layers "B.Cu" "B.Paste" "B.Mask") (roundrect_rratio 0.25)
       (net 1 "+5V") (pinfunction "Vref") (pintype "power_in"))
-    (pad "2" smd rect (at -2.725 0.635 180) (size 2 0.6) (layers "B.Cu" "B.Paste" "B.Mask")
+    (pad "2" smd roundrect (at -2.475 0.635 180) (size 1.95 0.6) (layers "B.Cu" "B.Paste" "B.Mask") (roundrect_rratio 0.25)
       (net 6 "Net-(U1-OUT)") (pinfunction "IN+") (pintype "input"))
-    (pad "3" smd rect (at -2.725 -0.635 180) (size 2 0.6) (layers "B.Cu" "B.Paste" "B.Mask")
+    (pad "3" smd roundrect (at -2.475 -0.635 180) (size 1.95 0.6) (layers "B.Cu" "B.Paste" "B.Mask") (roundrect_rratio 0.25)
       (net 5 "GND") (pinfunction "IN-") (pintype "input"))
-    (pad "4" smd rect (at -2.725 -1.905 180) (size 2 0.6) (layers "B.Cu" "B.Paste" "B.Mask")
+    (pad "4" smd roundrect (at -2.475 -1.905 180) (size 1.95 0.6) (layers "B.Cu" "B.Paste" "B.Mask") (roundrect_rratio 0.25)
       (net 5 "GND") (pinfunction "Vss") (pintype "power_in"))
-    (pad "5" smd rect (at 2.725 -1.905 180) (size 2 0.6) (layers "B.Cu" "B.Paste" "B.Mask")
+    (pad "5" smd roundrect (at 2.475 -1.905 180) (size 1.95 0.6) (layers "B.Cu" "B.Paste" "B.Mask") (roundrect_rratio 0.25)
       (net 3 "CE") (pinfunction "~{CS}/SHDN") (pintype "input"))
-    (pad "6" smd rect (at 2.725 -0.635 180) (size 2 0.6) (layers "B.Cu" "B.Paste" "B.Mask")
+    (pad "6" smd roundrect (at 2.475 -0.635 180) (size 1.95 0.6) (layers "B.Cu" "B.Paste" "B.Mask") (roundrect_rratio 0.25)
       (net 4 "MISO") (pinfunction "Dout") (pintype "output"))
-    (pad "7" smd rect (at 2.725 0.635 180) (size 2 0.6) (layers "B.Cu" "B.Paste" "B.Mask")
+    (pad "7" smd roundrect (at 2.475 0.635 180) (size 1.95 0.6) (layers "B.Cu" "B.Paste" "B.Mask") (roundrect_rratio 0.25)
       (net 2 "CLK") (pinfunction "CLK") (pintype "input"))
-    (pad "8" smd rect (at 2.725 1.905 180) (size 2 0.6) (layers "B.Cu" "B.Paste" "B.Mask")
+    (pad "8" smd roundrect (at 2.475 1.905 180) (size 1.95 0.6) (layers "B.Cu" "B.Paste" "B.Mask") (roundrect_rratio 0.25)
       (net 1 "+5V") (pinfunction "Vdd") (pintype "power_in"))
-    (model "${KICAD6_3DMODEL_DIR}/Package_SO.3dshapes/PowerIntegrations_SO-8.wrl"
+    (model "${KICAD6_3DMODEL_DIR}/Package_SO.3dshapes/SOIC-8_3.9x4.9mm_P1.27mm.wrl"
       (offset (xyz 0 0 0))
       (scale (xyz 1 1 1))
