File: RH_BreakLever_FreeJoy/RH_BreakLever_FreeJoy.kicad_sch (KiCad schematic)
At the start: 3 parts, among them J1 Conn_01x05, U1 SS495A, U2 MCP3201

Commit message: updated a footprint on Break-lever design for footprint naming.
Parts:
- U2: footprint Package_SO:PowerIntegrations_SO-8 -> Package_SO:SOIC-8_3.9x4.9mm_P1.27mm
Changed lines of the file:
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@@
       (effects (font (size 1.27 1.27)) (justify left))
     )
-    (property "Footprint" "Package_SO:PowerIntegrations_SO-8" (at 129.54 39.37 0)
+    (property "Footprint" "Package_SO:SOIC-8_3.9x4.9mm_P1.27mm" (at 129.54 39.37 0)
       (effects (font (size 1.27 1.27)) hide)
     )
