File: RH_GripLogicBoard_FreeJoy/RH_GripLogicBoard_FreeJoy.kicad_pcb (KiCad board)
At the start: 2 copper layers, 40.3 x 52.6 mm, 23 parts, among them J1 Conn_01x06, J2 Conn_01x06, J3 Conn_01x06, J4 Conn_01x02, J5 Conn_01x02, J6 Conn_01x07, J7 Conn_01x02, J8 Conn_01x02, U1 74HC165, U2 74HC165

Commit message: fixed mistake in Grip logic pcb's
Parts:
- J1: footprint Connector_JST:JST_XH_B8B-XH-A_1x08_P2.50mm_Vertical -> Connector_JST:JST_XH_B7B-XH-A_1x07_P2.50mm_Vertical
Connections:
- J1 pad 5: CE -> CE_GRIP
- J1 pad 6: Data_Head -> CE_HEAD
- J2 pad 4: Data_Head -> MISO
- J2 pad 5: CE -> CE_HEAD
- J3 pad 4: Data_Breaklever -> MISO
- U1 pad 1: CE -> CE_GRIP
- U2 pad 1: CE -> CE_GRIP
Routing:
- net CE_HEAD: track 0.00 -> 76.5 mm
- net MISO: track 24.2 -> 94.9 mm
- net CE: track 66.6 -> 0.00 mm, vias 1 -> 0
- net Data_Head: track 61.0 -> 0.00 mm
- net Data_Breaklever: track 53.4 -> 0.00 mm
- net CE_GRIP: track 0.00 -> 48.7 mm
